File: MOT_Photodiode.kicad_pcb (KiCad board)
At the start: 2 copper layers, 32 x 25 mm, 18 parts, among them J1 Supply, J2 output, J3 photodiode, U1 LT3032-12, U2 ADA4898-1YRDZ

Commit message: Bump version to 1.1.1
Other:
- board text added: "MOT_photodiode 1.1.1 Design: T. Preuschoff Date: 2025-02 https://github.com/ TU-Darmstadt-APQ"
- board text removed: "MOT_photodiode 1.1.0 Design: T. Preuschoff Date: 2025-02 https://github.com/ TU-Darmstadt-APQ"
Changed lines of the file:
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@@
 		)
 	)
-	(gr_text "MOT_photodiode 1.1.0\nDesign: T. Preuschoff\nDate: 2025-02\nhttps://github.com/\nTU-Darmstadt-APQ"
+	(gr_text "MOT_photodiode 1.1.1\nDesign: T. Preuschoff\nDate: 2025-02\nhttps://github.com/\nTU-Darmstadt-APQ"
 		(at 131.25 101.25 270)
 		(layer "B.SilkS")

Commit message: More version bumping to 1.1.1
Other:
- board text added: "MOT_photodiode 1.1.1 Design: T. Preuschoff Date: 2025-06 https://github.com/ TU-Darmstadt-APQ"
- board text removed: "MOT_photodiode 1.1.1 Design: T. Preuschoff Date: 2025-02 https://github.com/ TU-Darmstadt-APQ"
Changed lines of the file:
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@@
 	(title_block
 		(title "MOT Photodiode")
-		(date "2025-02-27")
-		(rev "1.1.0")
+		(date "2025-06-24")
+		(rev "1.1.1")
 		(company "Atoms Photons Quanta")
 		(comment 1 "and Tilman Preuschoff")
@@
 		)
 	)
-	(gr_text "MOT_photodiode 1.1.1\nDesign: T. Preuschoff\nDate: 2025-02\nhttps://github.com/\nTU-Darmstadt-APQ"
+	(gr_text "MOT_photodiode 1.1.1\nDesign: T. Preuschoff\nDate: 2025-06\nhttps://github.com/\nTU-Darmstadt-APQ"
 		(at 131.25 101.25 270)
 		(layer "B.SilkS")
